File: KiCad/L1B1/Unified-Daughterboard.sch (KiCad schematic (older format))
At the start: 10 parts, among them J2 SM04B-SRSS-TB(LF)(SN)

Commit message: Make the db
Parts:
- removed D?: PRTR5V0U2X,215, Package_TO_SOT_SMD:SOT-143, symbol Power_Protection:PRTR5V0U2X
- added U1: PRTR5V0U2X, random-keyboard-parts:SOT143B, symbol random-keyboard-parts:PRTR5V0U2X
- J1: renamed from J?; footprint (none) -> locallib:EXG.1B.305.HLN
Connections:
- net DN: now also U1.3 (IO2)
- net DP: now also U1.2 (IO1)
- net GNDPWR: now also U1.1 (GND)
- net VBUS: now also U1.4 (VCC)
Changed lines of the file:
@@
 L power:GNDPWR #PWR0112
 U 1 1 5E78F900
-P 4175 2375
-F 0 "#PWR0112" H 4175 2175 50  0001 C CNN
-F 1 "GNDPWR" H 4175 2275 15  0000 C CNN
-F 2 "" H 4175 2325 50  0001 C CNN
-F 3 "" H 4175 2325 50  0001 C CNN
-	1    4175 2375
+P 3725 2200
+F 0 "#PWR0112" H 3725 2000 50  0001 C CNN
+F 1 "GNDPWR" H 3725 2100 15  0000 C CNN
+F 2 "" H 3725 2150 50  0001 C CNN
+F 3 "" H 3725 2150 50  0001 C CNN
+	1    3725 2200
 	1    0    0    -1
 $EndComp
 $Comp
-L power:VBUS #PWR?
+L power:VBUS #PWR0101
 U 1 1 60775474
-P 4175 1375
-F 0 "#PWR?" H 4175 1225 50  0001 C CNN
-F 1 "VBUS" H 4175 1525 30  0000 C CNN
-F 2 "" H 4175 1375 50  0001 C CNN
-F 3 "" H 4175 1375 50  0001 C CNN
-	1    4175 1375
+P 4575 1825
+F 0 "#PWR0101" H 4575 1675 50  0001 C CNN
+F 1 "VBUS" H 4575 1975 30  0000 C CNN
+F 2 "" H 4575 1825 50  0001 C CNN
+F 3 "" H 4575 1825 50  0001 C CNN
+	1    4575 1825
 	1    0    0    -1
 $EndComp
-Text GLabel 4675 1875 2    50   Input ~ 0
+Text GLabel 4475 2125 2    50   Input ~ 0
 DN
-Text GLabel 3675 1875 0    50   Input ~ 0
+Text GLabel 3800 1650 0    50   Input ~ 0
 DP
-$Comp
-L Power_Protection:PRTR5V0U2X D?
-U 1 1 6076CFE9
-P 4175 1875
-F 0 "D?" H 4525 2200 50  0000 L CNN
-F 1 "PRTR5V0U2X,215" H 4525 2125 50  0000 L CNN
-F 2 "Package_TO_SOT_SMD:SOT-143" H 4235 1875 50  0001 C CNN
-F 3 "https://assets.nexperia.com/documents/data-sheet/PRTR5V0U2X.pdf" H 4235 1875 50  0001 C CNN
-	1    4175 1875
-	1    0    0    -1
-$EndComp
 Wire Wire Line
 	1425 2150 1750 2150
@@
 DP
 $Comp
-L power:GND #PWR?
+L power:GND #PWR0102
 U 1 1 6077D30C
 P 1750 2450
-F 0 "#PWR?" H 1750 2200 50  0001 C CNN
+F 0 "#PWR0102" H 1750 2200 50  0001 C CNN
 F 1 "GND" H 1755 2277 50  0000 C CNN
 F 2 "" H 1750 2450 50  0001 C CNN
@@
 	1750 2450 1425 2450
 $Comp
-L Connector_Generic:Conn_01x06 J?
+L Connector_Generic:Conn_01x06 J1
 U 1 1 6076A9E3
 P 1225 2350
-F 0 "J?" H 1143 2767 50  0000 C CNN
+F 0 "J1" H 1143 2767 50  0000 C CNN
 F 1 "EXG.1B.305.HLN" H 1143 2676 50  0000 C CNN
-F 2 "" H 1225 2350 50  0001 C CNN
+F 2 "locallib:EXG.1B.305.HLN" H 1225 2350 50  0001 C CNN
 F 3 "~" H 1225 2350 50  0001 C CNN
 	1    1225 2350
@@
 	1475 2550 1425 2550
 Connection ~ 1475 2650
+$Comp
+L random-keyboard-parts:PRTR5V0U2X U1
+U 1 1 60770E79
+P 4175 2075
+F 0 "U1" H 4175 2372 60  0000 C CNN
+F 1 "PRTR5V0U2X" H 4175 2266 60  0000 C CNN
+F 2 "random-keyboard-parts:SOT143B" H 4175 2075 60  0001 C CNN
+F 3 "" H 4175 2075 60  0001 C CNN
+	1    4175 2075
+	1    0    0    -1
+$EndComp
+Wire Wire Line
+	3725 2200 3725 2025
+Wire Wire Line
+	3725 2025 3875 2025
+Wire Wire Line
+	3800 1650 3800 2125
+Wire Wire Line
+	3800 2125 3875 2125
+Wire Wire Line
+	4575 1825 4575 2025
+Wire Wire Line
+	4575 2025 4475 2025
 $EndSCHEMATC
