File: KiCad/C3R/Unified-Daughterboard.kicad_pcb (KiCad board)
At the start: 2 copper layers, 18 x 16.5 mm, 13 parts, among them J1 TYPE-C-31-M12_13, J2 SM04B-SRSS-TB(LF)(SN), U1 TPD4E05U06DQAR

Commit message: Progress
Parts:
- removed G1: Unified-Daughterboard-Logo, Unified-Daughterboard-Logo:Unified-Daughterboard-Logo.pretty
- G2: footprint Unified-Daughterboard-Logo:Unified-Daughterboard-Name.pretty -> Unified-Daughterboard-Logo:Unified-Daughterboard-Name-NoID.pretty
Other:
- outline, holes or cut-outs redrawn
- board text added: "Ver. C3R"

Commit message: Create prod data
Parts:
- removed G2: Unified-Daughterboard-Name, Unified-Daughterboard-Logo:Unified-Daughterboard-Name-NoID.pretty
- moved D1 0.51 mm to (69.2, 66.9)
Routing:
- net VCC: track 16.3 -> 15.5 mm
Other:
- board text added: "Unified-DB Ver. C3R"
- board text removed: "Ver. C3R"
